File: PCB/Ark.kicad_sch (KiCad schematic)
At the start: 47 parts, among them P1 mode, P2 down, P3 up, SW1 EC12, SW2 EC12, SW3 EC12, SW4 EC12, SW5 EC12, SW6 EC12, SW7 EC12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

Commit message: Add files via upload
Parts:
- CP1: renamed from CPU1; footprint MyLibrary:2tht-5.08 -> MyLibrary:HUSG16M
- CP2: renamed from CPU2; footprint MyLibrary:2tht-5.08 -> MyLibrary:HUSG16M
- RC1, RC2, RC3, RC4: value 22 -> 22pf
Changed lines of the file:
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@@
       (effects (font (size 1.27 1.27)))
     )
-    (property "Value" "22" (at 181.61 74.93 90)
+    (property "Value" "22pf" (at 181.61 74.93 90)
       (effects (font (size 1.27 1.27)))
     )
@@
       (effects (font (size 1.27 1.27)))
     )
-    (property "Value" "22" (at 275.59 76.2 90)
+    (property "Value" "22pf" (at 275.59 76.2 90)
       (effects (font (size 1.27 1.27)))
     )
@@
   (symbol (lib_id "user:HUSG-16MHz") (at 273.05 62.23 0) (unit 1)
     (in_bom yes) (on_board yes) (dnp no)
-    (property "Reference" "CPU2" (at 279.4 62.865 0)
+    (property "Reference" "CP2" (at 279.4 62.865 0)
       (effects (font (size 1.27 1.27)) (justify left))
     )
@@
       (effects (font (size 1.27 1.27)))
     )
-    (property "Footprint" "MyLibrary:2tht-5.08" (at 273.05 62.23 0)
+    (property "Footprint" "MyLibrary:HUSG16M" (at 273.05 62.23 0)
       (effects (font (size 1.27 1.27)) hide)
     )
@@
       (project "Ark"
         (path "/33c2f9e4-7ccb-486c-ac6a-6f83bb66703d"
-          (reference "CPU2") (unit 1)
+          (reference "CP2") (unit 1)
         )
       )
@@
       (effects (font (size 1.27 1.27)))
     )
-    (property "Value" "22" (at 275.59 44.45 90)
+    (property "Value" "22pf" (at 275.59 44.45 90)
       (effects (font (size 1.27 1.27)))
     )
@@
       (effects (font (size 1.27 1.27)))
     )
-    (property "Value" "22" (at 181.61 43.18 90)
+    (property "Value" "22pf" (at 181.61 43.18 90)
       (effects (font (size 1.27 1.27)))
     )
@@
   (symbol (lib_name "HUSG-16MHz_1") (lib_id "user:HUSG-16MHz") (at 179.07 60.96 0) (unit 1)
     (in_bom yes) (on_board yes) (dnp no)
-    (property "Reference" "CPU1" (at 185.42 61.595 0)
+    (property "Reference" "CP1" (at 185.42 61.595 0)
       (effects (font (size 1.27 1.27)) (justify left))
     )
@@
       (effects (font (size 1.27 1.27)))
     )
-    (property "Footprint" "MyLibrary:2tht-5.08" (at 179.07 60.96 0)
+    (property "Footprint" "MyLibrary:HUSG16M" (at 179.07 60.96 0)
       (effects (font (size 1.27 1.27)) hide)
     )
@@
       (project "Ark"
         (path "/33c2f9e4-7ccb-486c-ac6a-6f83bb66703d"
-          (reference "CPU1") (unit 1)
-        )
-      )
+          (reference "CP1") (unit 1)
+        )
+      )

Commit message: Add files via upload
Parts:
- D1: renamed from 2281BS1; symbol 2281BS:2281BS_7seg*2 -> 2281BS:2281
Other:
- title: Ark.*~ Product -> ark.*~
- moved on the sheet: C1, C10, C11, C12, C13, C14, C15, C16, C2, C3, C4, C5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
